File: controller.brd (EAGLE design)
At the start: 39.3 x 41.1 mm, 33 parts, among them IC1 TM4C123[7,G]XXPM, U1 3.3V/150mA, Y1 CRYSTAL.3.2X2.5MM

Commit message: cleaned and updated files
Parts:
- removed LED1: (no value), Ilya_Teach:LED-0603
- added C13, C16: 2.2uF, SparkFun-Capacitors:0805
- added C14, C15: 0.1uF, microbuilder:_0603MP
- added J7: (no value), SparkFun-Connectors:1X02
- added PF0, PF3, PWR: (no value), Ilya_Teach:LED-0603
- added R6, R7: (no value), microbuilder:_0603MP
- added R8: 120, microbuilder:_0603MP
- added U2: MCP2551, SparkFun-IC-Comms:SO08
- added U3: 3.3V/150mA, SparkFun-IC-Power:SOT23-5
- LOGICPOWER, MOTORPOWER: device SparkFun-Connectors:1X02 -> SparkFun-Connectors:1X02@1
- MOTOR1, MOTOR2: device SparkFun-Connectors:1X02_2.54_SCREWTERM -> SparkFun-Connectors:1X02_2.54_SCREWTERM@1
- R4: value 100 -> 100R
- moved C10 4.49 mm to (9.91, 29.2), turned to 0 degrees
- moved Y1 2.72 mm to (34.5, 25.5), turned to 0 degrees
- moved R3 0.92 mm to (35.1, 30.7)
- moved R4 0.25 mm to (37.7, 30.7)
- moved R5 0.13 mm to (24.1, 38.0)
Connections:
- removed net N$25: IC1.58, J1.7
- removed net N$26: IC1.57, J1.8
- new net 5V: C15.2, C16.1, U2.3, U3.5
- new net CANH: J7.1, R8.1, U2.7
- new net CANL: J7.2, R8.2, U2.6
- new net N$5: PF0.C, R6.2
- new net N$7: PF3.C, R7.2
- new net PB4: IC1.58, J1.7, U2.4
- new net PB5: IC1.57, J1.8, U2.1
- new net PB6: IC1.1, U2.8
- net 12V: now also U3.1, U3.3
- net 3.3V: now also C13.1, C14.1, PWR.A, U2.5; no longer LED1.A
- net GND: now also C13.2, C14.2, C15.1, C16.2, R6.1, R7.1, U2.2, U3.2
- net N$51: now also PWR.C; no longer LED1.C
- net PF0: now also PF0.A
- net PF3: now also PF3.A
Routing:
- net PB5: track 0.00 -> 34.2 mm
- net PB4: track 0.00 -> 28.1 mm
- net 5V: track 0.00 -> 25.6 mm
- net PB6: track 0.00 -> 24.5 mm, vias 0 -> 1
- net 12V: track 37.7 -> 53.4 mm, vias 1 -> 2
- net CANL: track 0.00 -> 12.4 mm
- net N$25: track 11.7 -> 0.00 mm
- net N$26: track 10.8 -> 0.00 mm
- net PF0: track 0.00 -> 9.72 mm
- net CANH: track 0.00 -> 9.37 mm, vias 0 -> 1
- net 3.3V: track 135.5 -> 143.6 mm, vias 8 -> 9
- net PF3: track 0.00 -> 6.36 mm
- net N$2: track 12.2 -> 7.58 mm
- net N$7: track 0.00 -> 1.79 mm
- net N$5: track 0.00 -> 1.66 mm
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Other:
- board text added: "CANH"
- board text added: "CANL"
- board text added: "TM4C123GH6PM Simple DC Motor Control with TB6612FNG Rev 2 9 APR 2018"
- board text removed: "TM4C123GH6PM Simple DC Motor Control with TB6612FNG Rev 1 25 March 2019"
