File: controller.sch (EAGLE design)
At the start: 33 parts, among them IC1 TM4C123[7,G]XXPM, U1 3.3V/150mA, Y1 CRYSTAL.3.2X2.5MM

Commit message: cleaned and updated files
Parts:
- added C13, C16: 2.2uF, SparkFun-Capacitors:2.2UF-0805-25V-(+80/-20%)
- added C14, C15: 0.1uF, microbuilder:CAP_CERAMIC_0603MP
- added J7: (no value), SparkFun-Connectors:CONN_02
- added PF0, PF3: (no value), Ilya_Teach:LED0603
- added R6, R7: (no value), microbuilder:RESISTOR_0603MP
- added R8: 120, microbuilder:RESISTOR_0603MP
- added U2: MCP2551, SparkFun-IC-Comms:MCP2551
- added U3: 3.3V/150mA, SparkFun-IC-Power:V_REG_MIC52053.3V
- R4: value 100 -> 100R
- renumbered LED1 to PWR
Connections:
- removed net N$25: IC1.PB4, J1.7
- removed net N$26: IC1.PB5, J1.8
- new net 5V: C15.P$2, C16.1, U2.VDD, U3.OUT
- new net CANH: J7.1, R8.1, U2.CANH
- new net CANL: J7.2, R8.2, U2.CANL
- new net N$5: PF0.C, R6.2
- new net N$7: PF3.C, R7.2
- new net PB4: IC1.PB4, J1.7, U2.RXD
- new net PB5: IC1.PB5, J1.8, U2.TXD
- new net PB6: IC1.PB6, U2.RS
- net 12V: now also U3.EN, U3.IN
- net 3.3V: now also C13.1, C14.P$1, U2.VREF
- net GND: now also C13.2, C14.P$2, C15.P$1, C16.2, R6.1, R7.1, U2.VSS, U3.GND
- net PF0: now also PF0.A
- net PF3: now also PF3.A
